File: regulator_5v.kicad_sch (KiCad schematic)
At the start: 0 parts

Commit message: 5vreg
Parts:
- added C6: CIN, symbol Device:C
- added C7: COUT, symbol Device:C
- added D3: D_Schottky, symbol Device:D_Schottky
- added L1: L, symbol Device:L
- added U4: LM2596SX, Package_TO_SOT_SMD:TO-263-5_TabPin3, symbol Regulator_Linear:IFX25401TBV
Connections:
- new net: D3.1 (K), L1.1, U4.2 (VOUT)
- new net 5V: C7.1, L1.2, U4.4 (FB)
- new net BATT+: C6.1, U4.1 (VIN)
- new net GND: C6.2, C7.2, D3.2 (A), U4.3 (GND), U4.5 (EN)
