File: robot_pcb.kicad_sch (KiCad schematic)
At the start: 27 parts, among them J1 Raspberry_Pi_2_3, J10 Servo_TrayRelease, J2 Motor FL, J3 Motor FR, J4 Motor BL, J5 Motor BR, J6 TOF_Front, J7 UltraS_Side, J8 Servo_Grab, J9 Servo_Lift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

Commit message: Update robot_pcb.kicad_sch
Parts:
- added C17: CIN, symbol Device:C
- added C18: COUT, symbol Device:C
- added D4: D_Schottky, symbol Device:D_Schottky
- added L2: L, symbol Device:L
- added U5: LM2596SX, Package_TO_SOT_SMD:TO-263-5_TabPin3, symbol Regulator_Linear:IFX25401TBV
Connections:
- net 5V: now also C18.1, L2.2, U5.4 (FB)
- net GND: now also C17.2, C18.2, D4.2 (A), U5.3 (GND), U5.5 (EN)
- new net: D4.1 (K), L2.1, U5.2 (VOUT)
- new net BATT+: C17.1, U5.1 (VIN)
Other:
- note added: "5V REGULATOR"
- moved on the sheet: D1, D2, J10, J2, J3, J4, J5, J6, J7, J8, J9

Commit message: s
Parts:
- added R7: 2k, symbol Device:R
- added R8: 6.2k, symbol Device:R
- D4: value D_Schottky -> B340A; footprint (none) -> Diode_SMD:D_SMA
- L2: value L -> 47uH
- U5: value LM2596SX -> AP1501-50K5G-13
Connections:
- net 5V: now also R8.1; no longer U5.4 (FB)
- net GND: now also R7.1
- new net: R7.2, R8.2, U5.4 (FB)
Other:
- removed sheet 5V Regulator
Changed lines of the file:
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@@
 	)
 	(junction
+		(at 66.04 24.13)
+		(diameter 0)
+		(color 0 0 0 0)
+	)
+	(junction
 		(at 290.83 196.85)
 		(diameter 0)
@@
 	(wire
 		(pts
-			(xy 80.01 25.4) (xy 80.01 27.94)
+			(xy 147.32 124.46) (xy 149.86 124.46)
 		)
 		(stroke
@@
 	(wire
 		(pts
-			(xy 147.32 124.46) (xy 149.86 124.46)
+			(xy 151.13 58.42) (xy 153.67 58.42)
 		)
 		(stroke
@@
 	(wire
 		(pts
-			(xy 151.13 58.42) (xy 153.67 58.42)
+			(xy 31.75 25.4) (xy 43.18 25.4)
 		)
 		(stroke
@@
 	(wire
 		(pts
-			(xy 31.75 25.4) (xy 43.18 25.4)
+			(xy 255.27 66.04) (xy 265.43 66.04)
 		)
 		(stroke
@@
 	(wire
 		(pts
-			(xy 255.27 66.04) (xy 265.43 66.04)
+			(xy 231.14 49.53) (xy 231.14 48.26)
 		)
 		(stroke
@@
 	(wire
 		(pts
-			(xy 231.14 49.53) (xy 231.14 48.26)
+			(xy 66.04 24.13) (xy 66.04 19.05)
 		)
 		(stroke
@@
 	(wire
 		(pts
+			(xy 63.5 25.4) (xy 66.04 25.4)
+		)
+		(stroke
+			(width 0)
+			(type default)
+		)
+	)
+	(wire
+		(pts
 			(xy 323.85 39.37) (xy 323.85 40.64)
 		)
@@
 	(wire
 		(pts
-			(xy 63.5 25.4) (xy 80.01 25.4)
+			(xy 66.04 24.13) (xy 66.04 25.4)
 		)
 		(stroke
@@
 	(wire
 		(pts
+			(xy 80.01 24.13) (xy 80.01 27.94)
+		)
+		(stroke
+			(width 0)
+			(type default)
+		)
+	)
+	(wire
+		(pts
 			(xy 149.86 124.46) (xy 152.4 124.46)
 		)
@@
 	(wire
 		(pts
+			(xy 73.66 24.13) (xy 80.01 24.13)
+		)
+		(stroke
+			(width 0)
+			(type default)
+		)
+	)
+	(wire
+		(pts
 			(xy 290.83 195.58) (xy 290.83 196.85)
 		)
@@
 		(dnp no)
 		(property "Reference" "L2"
-			(at 76.2 23.622 90)
+			(at 76.2 25.908 90)
 			(effects
 				(font
@@
 			)
 		)
-		(property "Value" "L"
+		(property "Value" "47uH"
 			(at 76.2 29.464 90)
 			(effects
@@
 	)
 	(symbol
+		(lib_id "power:GND")
+		(at 73.66 19.05 90)
+		(unit 1)
+		(exclude_from_sim no)
+		(in_bom yes)
+		(on_board yes)
+		(dnp no)
+		(fields_autoplaced yes)
+		(property "Reference" "#PWR019"
+			(at 80.01 19.05 0)
+			(effects
+				(font
+					(size 1.27 1.27)
+				)
+				(hide yes)
+			)
+		)
+		(property "Value" "GND"
+			(at 77.47 19.0499 90)
+			(effects
+				(font
+					(size 1.27 1.27)
+				)
+				(justify right)
+			)
+		)
+		(property "Footprint" ""
+			(at 73.66 19.05 0)
+			(effects
+				(font
+					(size 1.27 1.27)
+				)
+				(hide yes)
+			)
+		)
+		(property "Datasheet" ""
+			(at 73.66 19.05 0)
+			(effects
+				(font
+					(size 1.27 1.27)
+				)
+				(hide yes)
+			)
+		)
+		(property "Description" "Power symbol creates a global label with name \"GND\" , ground"
+			(at 73.66 19.05 0)
+			(effects
+				(font
+					(size 1.27 1.27)
+				)
+				(hide yes)
+			)
+		)
+		(pin "1"
+		)
+		(instances
+			(project "robot_pcb"
+				(path "/2f56b371-1597-47e1-a48d-b7f69d342f77"
+					(reference "#PWR019")
+					(unit 1)
+				)
+			)
+		)
+	)
+	(symbol
 		(lib_id "Device:C")
 		(at 31.75 29.21 0)
@@
 	)
 	(symbol
+		(lib_id "Device:R")
+		(at 69.85 19.05 270)
+		(unit 1)
+		(exclude_from_sim no)
+		(in_bom yes)
+		(on_board yes)
+		(dnp no)
+		(property "Reference" "R7"
+			(at 69.85 19.05 90)
+			(effects
+				(font
+					(size 1.27 1.27)
+				)
+			)
+		)
+		(property "Value" "2k"
+			(at 69.85 21.336 90)
+			(effects
+				(font
+					(size 1.27 1.27)
+				)
+			)
+		)
+		(property "Footprint" ""
+			(at 69.85 17.272 90)
+			(effects
+				(font
+					(size 1.27 1.27)
+				)
+				(hide yes)
+			)
+		)
+		(property "Datasheet" "~"
+			(at 69.85 19.05 0)
+			(effects
+				(font
+					(size 1.27 1.27)
+				)
+				(hide yes)
+			)
+		)
+		(property "Description" "Resistor"
+			(at 69.85 19.05 0)
+			(effects
+				(font
+					(size 1.27 1.27)
+				)
+				(hide yes)
+			)
+		)
+		(pin "2"
+		)
+		(pin "1"
+		)
+		(instances
+			(project ""
+				(path "/2f56b371-1597-47e1-a48d-b7f69d342f77"
+					(reference "R7")
+					(unit 1)
+				)
+			)
+		)
+	)
+	(symbol
+		(lib_id "Device:R")
+		(at 69.85 24.13 270)
+		(unit 1)
+		(exclude_from_sim no)
+		(in_bom yes)
+		(on_board yes)
+		(dnp no)
+		(property "Reference" "R8"
+			(at 69.85 24.13 90)
+			(effects
+				(font
+					(size 1.27 1.27)
+				)
+			)
+		)
+		(property "Value" "6.2k"
+			(at 69.85 26.416 90)
+			(effects
+				(font
+					(size 1.27 1.27)
+				)
+			)
+		)
+		(property "Footprint" ""
+			(at 69.85 22.352 90)
+			(effects
+				(font
+					(size 1.27 1.27)
+				)
+				(hide yes)
+			)
+		)
+		(property "Datasheet" "~"
+			(at 69.85 24.13 0)
+			(effects
+				(font
+					(size 1.27 1.27)
+				)
+				(hide yes)
+			)
+		)
+		(property "Description" "Resistor"
+			(at 69.85 24.13 0)
+			(effects
+				(font
+					(size 1.27 1.27)
+				)
+				(hide yes)
+			)
+		)
+		(pin "2"
+		)
+		(pin "1"
+		)
+		(instances
+			(project "robot_pcb"
+				(path "/2f56b371-1597-47e1-a48d-b7f69d342f77"
+					(reference "R8")
+					(unit 1)
+				)
+			)
+		)
+	)
+	(symbol
 		(lib_id "Connector_Generic:Conn_01x04")
 		(at 250.19 219.71 270)
@@
 			)
 		)
-		(property "Value" "LM2596SX"
+		(property "Value" "AP1501-50K5G-13"
 			(at 53.34 20.32 0)
 			(effects
@@
 			)
 		)
-		(property "Value" "D_Schottky"
+		(property "Value" "B340A"
 			(at 68.58 32.7024 90)
 			(effects
@@
 			)
 		)
-		(property "Footprint" ""
+		(property "Footprint" "Diode_SMD:D_SMA"
 			(at 66.04 31.75 0)
 			(effects
@@
 				)
 			)
-		)
-	)
-	(sheet
-		(at 35.56 120.65)
-		(size 40.64 27.94)
-		(exclude_from_sim no)
-		(in_bom yes)
-		(on_board yes)
-		(dnp no)
-		(fields_autoplaced yes)
-		(stroke
-			(width 0.1524)
-			(type solid)
-		)
-		(fill
-			(color 0 0 0 0.0000)
-		)
-		(property "Sheetname" "5V Regulator"
-			(at 35.56 119.9384 0)
-			(effects
-				(font
-					(size 1.27 1.27)
-				)
-				(justify left bottom)
-			)
-		)
-		(property "Sheetfile" "regulator_5v.kicad_sch"
-			(at 35.56 149.1746 0)
-			(effects
-				(font
-					(size 1.27 1.27)
-				)
-				(justify left top)
-			)
-		)
-		(instances
-			(project "robot_pcb"
-				(path "/2f56b371-1597-47e1-a48d-b7f69d342f77"
-					(page "4")
-				)
-			)

Commit message: Update robot_pcb.kicad_sch
Parts:
- removed R7: 2k, symbol Device:R
- removed R8: 6.2k, symbol Device:R
Connections:
- net 5V: now also U5.4 (FB)
Changed lines of the file:
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@@
 	)
 	(junction
-		(at 66.04 24.13)
-		(diameter 0)
-		(color 0 0 0 0)
-	)
-	(junction
 		(at 290.83 196.85)
 		(diameter 0)
@@
 	(wire
 		(pts
-			(xy 66.04 24.13) (xy 66.04 19.05)
-		)
-		(stroke
-			(width 0)
-			(type default)
-		)
-	)
-	(wire
-		(pts
 			(xy 308.61 39.37) (xy 323.85 39.37)
 		)
@@
 	(wire
 		(pts
-			(xy 63.5 25.4) (xy 66.04 25.4)
+			(xy 63.5 24.13) (xy 80.01 24.13)
 		)
 		(stroke
@@
 	(wire
 		(pts
-			(xy 66.04 24.13) (xy 66.04 25.4)
-		)
-		(stroke
-			(width 0)
-			(type default)
-		)
-	)
-	(wire
-		(pts
 			(xy 205.74 39.37) (xy 218.44 39.37)
 		)
@@
 	(wire
 		(pts
-			(xy 290.83 49.53) (xy 290.83 50.8)
+			(xy 63.5 24.13) (xy 63.5 25.4)
 		)
 		(stroke
@@
 	(wire
 		(pts
-			(xy 193.04 39.37) (xy 193.04 40.64)
+			(xy 290.83 49.53) (xy 290.83 50.8)
 		)
 		(stroke
@@
 	(wire
 		(pts
-			(xy 293.37 195.58) (xy 293.37 196.85)
+			(xy 193.04 39.37) (xy 193.04 40.64)
 		)
 		(stroke
@@
 	(wire
 		(pts
-			(xy 73.66 24.13) (xy 80.01 24.13)
+			(xy 293.37 195.58) (xy 293.37 196.85)
 		)
 		(stroke
@@
 	)
 	(symbol
-		(lib_id "power:GND")
-		(at 73.66 19.05 90)
-		(unit 1)
-		(exclude_from_sim no)
-		(in_bom yes)
-		(on_board yes)
-		(dnp no)
-		(fields_autoplaced yes)
-		(property "Reference" "#PWR019"
-			(at 80.01 19.05 0)
-			(effects
-				(font
-					(size 1.27 1.27)
-				)
-				(hide yes)
-			)
-		)
-		(property "Value" "GND"
-			(at 77.47 19.0499 90)
-			(effects
-				(font
-					(size 1.27 1.27)
-				)
-				(justify right)
-			)
-		)
-		(property "Footprint" ""
-			(at 73.66 19.05 0)
-			(effects
-				(font
-					(size 1.27 1.27)
-				)
-				(hide yes)
-			)
-		)
-		(property "Datasheet" ""
-			(at 73.66 19.05 0)
-			(effects
-				(font
-					(size 1.27 1.27)
-				)
-				(hide yes)
-			)
-		)
-		(property "Description" "Power symbol creates a global label with name \"GND\" , ground"
-			(at 73.66 19.05 0)
-			(effects
-				(font
-					(size 1.27 1.27)
-				)
-				(hide yes)
-			)
-		)
-		(pin "1"
-		)
-		(instances
-			(project "robot_pcb"
-				(path "/2f56b371-1597-47e1-a48d-b7f69d342f77"
-					(reference "#PWR019")
-					(unit 1)
-				)
-			)
-		)
-	)
-	(symbol
 		(lib_id "Device:C")
 		(at 31.75 29.21 0)
@@
 					(unit 1)
 				)
-			)
-		)
-	)
-	(symbol
-		(lib_id "Device:R")
-		(at 69.85 19.05 270)
-		(unit 1)
-		(exclude_from_sim no)
-		(in_bom yes)
-		(on_board yes)
-		(dnp no)
-		(property "Reference" "R7"
-			(at 69.85 19.05 90)
-			(effects
-				(font
-					(size 1.27 1.27)
-				)
-			)
-		)
-		(property "Value" "2k"
-			(at 69.85 21.336 90)
-			(effects
-				(font
-					(size 1.27 1.27)
-				)
-			)
-		)
-		(property "Footprint" ""
-			(at 69.85 17.272 90)
-			(effects
-				(font
-					(size 1.27 1.27)
-				)
-				(hide yes)
-			)
-		)
-		(property "Datasheet" "~"
-			(at 69.85 19.05 0)
-			(effects
-				(font
-					(size 1.27 1.27)
-				)
-				(hide yes)
-			)
-		)
-		(property "Description" "Resistor"
-			(at 69.85 19.05 0)
-			(effects
-				(font
-					(size 1.27 1.27)
-				)
-				(hide yes)
-			)
-		)
-		(pin "2"
-		)
-		(pin "1"
-		)
-		(instances
-			(project ""
-				(path "/2f56b371-1597-47e1-a48d-b7f69d342f77"
-					(reference "R7")
-					(unit 1)
-				)
-			)
-		)
-	)
-	(symbol
-		(lib_id "Device:R")
-		(at 69.85 24.13 270)
-		(unit 1)
-		(exclude_from_sim no)
-		(in_bom yes)
-		(on_board yes)
-		(dnp no)
-		(property "Reference" "R8"
-			(at 69.85 24.13 90)
-			(effects
-				(font
-					(size 1.27 1.27)
-				)
-			)
-		)
-		(property "Value" "6.2k"
-			(at 69.85 26.416 90)
-			(effects
-				(font
-					(size 1.27 1.27)
-				)
-			)
-		)
-		(property "Footprint" ""
-			(at 69.85 22.352 90)
-			(effects
-				(font
-					(size 1.27 1.27)
-				)
-				(hide yes)
-			)
-		)
-		(property "Datasheet" "~"
-			(at 69.85 24.13 0)
-			(effects
-				(font
-					(size 1.27 1.27)
-				)
-				(hide yes)
-			)
-		)
-		(property "Description" "Resistor"
-			(at 69.85 24.13 0)
-			(effects
-				(font
-					(size 1.27 1.27)
-				)
-				(hide yes)
-			)
-		)
-		(pin "2"
-		)
-		(pin "1"
-		)
-		(instances
-			(project "robot_pcb"
-				(path "/2f56b371-1597-47e1-a48d-b7f69d342f77"
-					(reference "R8")
-					(unit 1)
-				)

Commit message: Update robot_pcb.kicad_sch
Parts:
- C17: value CIN -> 680uF
- C18: value COUT -> 220uF
- D4: value B340A -> 1N5824
- L2: value 47uH -> 33uH
- U5: value AP1501-50K5G-13 -> LM2596DP-5.0
Changed lines of the file:
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@@
 	(wire
 		(pts
-			(xy 80.01 27.94) (xy 76.2 27.94)
-		)
-		(stroke
-			(width 0)
-			(type default)
-		)
-	)
-	(wire
-		(pts
 			(xy 218.44 49.53) (xy 231.14 49.53)
 		)
@@
 			)
 		)
-		(property "Value" "47uH"
+		(property "Value" "33uH"
 			(at 76.2 29.464 90)
 			(effects
@@
 			)
 		)
-		(property "Value" "COUT"
+		(property "Value" "220uF"
 			(at 87.63 33.0199 0)
 			(effects
@@
 			)
 		)
-		(property "Value" "CIN"
+		(property "Value" "680uF"
 			(at 35.56 30.4799 0)
 			(effects
@@
 			)
 		)
-		(property "Value" "AP1501-50K5G-13"
+		(property "Value" "LM2596DP-5.0"
 			(at 53.34 20.32 0)
 			(effects
@@
 			)
 		)
-		(property "Datasheet" ""
+		(property "Datasheet" "https://www.lcsc.com/datasheet/C77782.pdf"
 			(at 55.626 43.434 0)
 			(effects
@@
 			)
 		)
-		(property "Value" "B340A"
+		(property "Value" "1N5824"
 			(at 68.58 32.7024 90)
 			(effects

Commit message: Update robot_pcb.kicad_sch
Parts:
- U5: value LM2596DP-5.0 -> LM2596R-5.0
Changed lines of the file:
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@@
 			)
 		)
-		(property "Value" "LM2596DP-5.0"
+		(property "Value" "LM2596R-5.0"
 			(at 53.34 20.32 0)
 			(effects

Commit message: Update robot_pcb.kicad_sch
Parts:
- C17: LCSC (none) -> C5221838
- C18: LCSC (none) -> C190724
Changed lines of the file:
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@@
+			)
+		)
+		(property "LCSC" "C190724"
+			(at 83.82 31.75 0)
+			(effects
+				(font
+					(size 1.27 1.27)
+				)
+				(hide yes)
 			)
 		)
@@
 			(at 31.75 29.21 0)
 			(effects
+				(font
+					(size 1.27 1.27)
+				)
+				(hide yes)
+			)
+		)
+		(property "LCSC" "C5221838"
+			(at 31.75 29.21 0)
+			(effects

Commit message: Update robot_pcb.kicad_sch
Parts:
- removed C17: 680uF, symbol Device:C
- removed C18: 220uF, symbol Device:C
- added C19: 330uF, symbol Device:C_Polarized
- added C20: 1uF, symbol Device:C
- added C21: 680uF, symbol Device:C_Polarized
- added C22: 470uF, symbol Device:C_Polarized
- added C23: 220uF, symbol Device:C_Polarized
- added D3: 1N5820, symbol Device:D_Schottky
- added L1: 47uH, symbol Device:L
- added U4: XL1509-3.3, Package_SO:SOIC-8_3.9x4.9mm_P1.27mm, symbol Regulator_Switching:XL1509-3.3
Connections:
- net 5V: now also C23.1
- net BATT+: now also C20.1, C21.1, C22.1, U4.1 (VIN)
- net GND: now also C19.2, C20.2, C21.2, C22.2, C23.2, D3.2 (A), U4.4 (~{EN}), U4.5 (GND), U4.6 (GND), U4.7 (GND), U4.8 (GND)
- new net: D3.1 (K), L1.1, U4.2 (OUT)
- new net 3V3: C19.1, L1.2, U4.3 (FB)
Other:
- note added: "3V3 REGULATOR"

Commit message: 3v3 done
Other:
- removed sheet 3.3V Regulator
Changed lines of the file:
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@@
-	)
-	(sheet
-		(at 35.56 157.48)
-		(size 40.64 27.94)
-		(exclude_from_sim no)
-		(in_bom yes)
-		(on_board yes)
-		(dnp no)
-		(fields_autoplaced yes)
-		(stroke
-			(width 0.1524)
-			(type solid)
-		)
-		(fill
-			(color 0 0 0 0.0000)
-		)
-		(property "Sheetname" "3.3V Regulator"
-			(at 35.56 156.7684 0)
-			(effects
-				(font
-					(size 1.27 1.27)
-				)
-				(justify left bottom)
-			)
-		)
-		(property "Sheetfile" "regulator_3v3.kicad_sch"
-			(at 35.56 186.0046 0)
-			(effects
-				(font
-					(size 1.27 1.27)
-				)
-				(justify left top)
-			)
-		)
-		(instances
-			(project "robot_pcb"
-				(path "/2f56b371-1597-47e1-a48d-b7f69d342f77"
-					(page "5")
-				)
-			)
-		)
 	)
 	(sheet
@@
 	)
 	(sheet
-		(at 33.02 96.52)
+		(at 40.64 194.31)
 		(size 40.64 27.94)
 		(exclude_from_sim no)
@@
 		)
 		(property "Sheetname" "12V Regulator"
-			(at 33.02 95.8084 0)
+			(at 40.64 193.5984 0)
 			(effects
 				(font
@@
 		)
 		(property "Sheetfile" "regulator_12v.kicad_sch"
-			(at 33.02 125.0446 0)
+			(at 40.64 222.8346 0)
 			(effects
 				(font
