File: regulators.kicad_sch (KiCad schematic)
At the start: 99 parts, among them IC1 IAUCN04S7L028ATMA1, Q6 Si7149DP, Q7 CSD17577Q3A, Q8 CSD17313Q2, Q9 CSD17578Q3A, U19 TPS611781RNWR, U20 XLM51772RHAR, U3 AP64501SP-13, U6 AP64501SP-13, U7 AP64501SP-13

Commit message: added lcsc part numbers for non trivial 12v components
Parts:
- C102: LCSC (none) -> C347564
- C104, C111, C112: LCSC (none) -> C2162042
- IC1: LCSC (none) -> C29536843
- L6: LCSC (none) -> C19191623
- Q7: LCSC (none) -> C201632
- Q8: LCSC (none) -> C2863837
- Q9: LCSC (none) -> C205986
- R67: LCSC (none) -> C2479048
- U20: LCSC (none) -> C41383743
Changed lines of the file:
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@@
 			)
 		)
+		(property "LCSC" "C41383743"
+			(at 217.17 228.6 0)
+			(effects
+				(font
+					(size 1.27 1.27)
+				)
+				(hide yes)
+			)
+		)
 		(pin "3"
 		)
@@
 			)
 		)
+		(property "LCSC" "C2162042"
+			(at 337.82 175.26 0)
+			(effects
+				(font
+					(size 1.27 1.27)
+				)
+				(hide yes)
+			)
+		)
 		(pin "2"
 		)
@@
 			)
 		)
+		(property "LCSC" "C347564"
+			(at 200.66 177.8 0)
+			(effects
+				(font
+					(size 1.27 1.27)
+				)
+				(hide yes)
+			)
+		)
 		(pin "2"
 		)
@@
 			)
 		)
+		(property "LCSC" "C205986"
+			(at 284.48 176.53 0)
+			(effects
+				(font
+					(size 1.27 1.27)
+				)
+				(hide yes)
+			)
+		)
 		(pin "5"
 		)
@@
 			)
 		)
+		(property "LCSC" "C2162042"
+			(at 325.12 175.26 0)
+			(effects
+				(font
+					(size 1.27 1.27)
+				)
+				(hide yes)
+			)
+		)
 		(pin "2"
 		)
@@
 			)
 		)
+		(property "LCSC" "C201632"
+			(at 236.22 176.53 0)
+			(effects
+				(font
+					(size 1.27 1.27)
+				)
+				(hide yes)
+			)
+		)
 		(pin "2"
 		)
@@
 			)
 		)
+		(property "LCSC" "C2479048"
+			(at 247.65 190.5 90)
+			(effects
+				(font
+					(size 1.27 1.27)
+				)
+				(hide yes)
+			)
+		)
 		(pin "1"
 		)
@@
 			)
 		)
+		(property "LCSC" "C2863837"
+			(at 236.22 203.2 0)
+			(effects
+				(font
+					(size 1.27 1.27)
+				)
+				(hide yes)
+			)
+		)
 		(pin "7"
 		)
@@
 			)
 		)
+		(property "LCSC" "C29536843"
+			(at 270.51 199.39 0)
+			(effects
+				(font
+					(size 1.27 1.27)
+				)
+				(hide yes)
+			)
+		)
 		(pin "3"
 		)
@@
 			)
 		)
+		(property "LCSC" "C19191623"
+			(at 265.43 190.5 90)
+			(effects
+				(font
+					(size 1.27 1.27)
+				)
+				(hide yes)
+			)
+		)
 		(pin "2"
 		)
@@
 			)
 		)
+		(property "LCSC" "C41383743"
+			(at 86.36 194.31 0)
+			(effects
+				(font
+					(size 1.27 1.27)
+				)
+				(hide yes)
+			)
+		)
 		(pin "3"
 		)
@@
 			(at 350.52 175.26 0)
 			(effects
+				(font
+					(size 1.27 1.27)
+				)
+				(hide yes)
+			)
+		)
+		(property "LCSC" "C2162042"
+			(at 350.52 175.26 0)
+			(effects

Commit message: lcsc numbers for other regulators
Parts:
- U3, U6, U7: LCSC (none) -> C2071517
Changed lines of the file:
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@@
 			)
 		)
-		(property "LCSC" ""
+		(property "LCSC" "C2071517"
 			(at 58.42 22.86 0)
 			(effects
@@
 			)
 		)
-		(property "LCSC" ""
+		(property "LCSC" "C2071517"
 			(at 58.42 111.76 0)
 			(effects
@@
 			)
 		)
-		(property "LCSC" ""
+		(property "LCSC" "C2071517"
 			(at 58.42 67.31 0)
 			(effects

Commit message: probably should have checked clearance
Parts:
- IC1: footprint IAUC120N06S5N011ATMA1 -> Dry_Lettuce:IAUC120N06S5N011ATMA1
Changed lines of the file:
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@@
 			)
 		)
-		(property "Footprint" "IAUC120N06S5N011ATMA1"
+		(property "Footprint" "Dry_Lettuce:IAUC120N06S5N011ATMA1"
 			(at 292.1 294.31 0)
 			(effects

Commit message: more lcsc
Parts:
- C109, C110, C86: LCSC (none) -> C1525
- C17, C42, C45: LCSC (none) -> C315248
- C84, C95, C96: LCSC (none) -> C309062
- C90: LCSC (none) -> C107147
- C92, R59: LCSC (none) -> C138687
- R18: LCSC (none) -> C25759
- R19: LCSC (none) -> C852490
- R20, R23: LCSC (none) -> C163478
- R21: LCSC (none) -> C5581335
- R22: LCSC (none) -> C852893
- R24: LCSC (none) -> C26956
- R25: value 115.8k -> 105k; LCSC (none) -> C171671
- R26: value 22.1k -> 20k; LCSC (none) -> C93942
- R60: LCSC (none) -> C13315
Connections:
- net 12V_COMP_MID renamed 3V3_COMP_MID
Changed lines of the file:
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@@
 		)
 	)
-	(label "12V_COMP_MID"
+	(label "3V3_COMP_MID"
 		(at 69.85 87.63 0)
 		(effects
@@
 			)
 		)
-		(property "LCSC" ""
+		(property "LCSC" "C163478"
 			(at 100.33 43.18 0)
 			(effects
@@
 			)
 		)
-		(property "LCSC" ""
+		(property "LCSC" "C852490"
 			(at 100.33 33.02 0)
 			(effects
@@
 			)
 		)
+		(property "LCSC" "C13315"
+			(at 300.99 64.77 0)
+			(effects
+				(font
+					(size 1.27 1.27)
+				)
+				(hide yes)
+			)
+		)
 		(pin "1"
 		)
@@
 			)
 		)
-		(property "LCSC" ""
+		(property "LCSC" "C315248"
 			(at 31.75 30.48 0)
 			(effects
@@
 			)
 		)
+		(property "LCSC" "C1525"
+			(at 205.74 245.11 0)
+			(effects
+				(font
+					(size 1.27 1.27)
+				)
+				(hide yes)
+			)
+		)
 		(pin "1"
 		)
@@
 			)
 		)
+		(property "LCSC" "C309062"
+			(at 177.8 38.1 0)
+			(effects
+				(font
+					(size 1.27 1.27)
+				)
+				(hide yes)
+			)
+		)
 		(pin "1"
 		)
@@
 			)
 		)
+		(property "LCSC" "C107147"
+			(at 281.94 64.77 0)
+			(effects
+				(font
+					(size 1.27 1.27)
+				)
+				(hide yes)
+			)
+		)
 		(pin "2"
 		)
@@
 			)
 		)
-		(property "LCSC" ""
+		(property "LCSC" "C315248"
 			(at 31.75 119.38 0)
 			(effects
@@
 			)
 		)
-		(property "LCSC" ""
+		(property "LCSC" "C26956"
 			(at 69.85 127 0)
 			(effects
@@
 			)
 		)
+		(property "LCSC" "C138687"
+			(at 254 63.5 0)
+			(effects
+				(font
+					(size 1.27 1.27)
+				)
+				(hide yes)
+			)
+		)
 		(pin "2"
 		)
@@
 			)
 		)
-		(property "Value" "22.1k"
+		(property "Value" "20k"
 			(at 102.87 133.3499 0)
 			(effects
@@
 			)
 		)
-		(property "LCSC" ""
+		(property "LCSC" "C93942"
 			(at 100.33 132.08 0)
 			(effects
@@
 			)
 		)
-		(property "LCSC" ""
+		(property "LCSC" "C25759"
 			(at 69.85 38.1 0)
 			(effects
@@
 			)
 		)
-		(property "LCSC" ""
+		(property "LCSC" "C315248"
 			(at 31.75 74.93 0)
 			(effects
@@
 			)
 		)
+		(property "LCSC" "C309062"
+			(at 166.37 38.1 0)
+			(effects
+				(font
+					(size 1.27 1.27)
+				)
+				(hide yes)
+			)
+		)
 		(pin "1"
 		)
@@
 			)
 		)
-		(property "LCSC" ""
+		(property "LCSC" "C852893"
 			(at 100.33 77.47 0)
 			(effects
@@
 			)
 		)
-		(property "Datasheet" ""
+		(property "Datasheet" "https://www.diodes.com/assets/Datasheets/AP64501.pdf"
 			(at 58.42 111.76 0)
 			(effects
@@
 			)
 		)
+		(property "LCSC" "C138687"
+			(at 269.24 64.77 0)
+			(effects
+				(font
+					(size 1.27 1.27)
+				)
+				(hide yes)
+			)
+		)
 		(pin "1"
 		)
@@
 			)
 		)
+		(property "LCSC" "C1525"
+			(at 193.04 242.57 0)
+			(effects
+				(font
+					(size 1.27 1.27)
+				)
+				(hide yes)
+			)
+		)
 		(pin "1"
 		)
@@
 			)
 		)
+		(property "LCSC" "C1525"
+			(at 257.81 50.8 0)
+			(effects
+				(font
+					(size 1.27 1.27)
+				)
+				(hide yes)
+			)
+		)
 		(pin "2"
 		)
@@
 			)
 		)
-		(property "Value" "115.8k"
+		(property "Value" "105k"
 			(at 101.854 123.952 0)
 			(effects
@@
 			)
 		)
-		(property "LCSC" ""
+		(property "LCSC" "C171671"
 			(at 100.33 121.92 0)
 			(effects
@@
 			)
 		)
-		(property "LCSC" ""
+		(property "LCSC" "C5581335"
 			(at 69.85 82.55 0)
 			(effects
@@
 			)
 		)
+		(property "LCSC" "C309062"
+			(at 189.23 38.1 0)
+			(effects
+				(font
+					(size 1.27 1.27)
+				)
+				(hide yes)
+			)
+		)
 		(pin "1"
 		)
@@
 			)
 		)
-		(property "LCSC" ""
+		(property "LCSC" "C163478"
 			(at 100.33 87.63 0)
 			(effects

Commit message: lcsc + changed footprint of a capacitor
Parts:
- C85: LCSC (none) -> C6119795
- C87: LCSC (none) -> C107031
- C88, C89, C97: LCSC (none) -> C138687
- C91, C93, C94: LCSC (none) -> C51205
- R56: LCSC (none) -> C114151
- R57: LCSC (none) -> C11537
- R58: LCSC (none) -> C25895
- R61: LCSC (none) -> C25921
Changed lines of the file:
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@@
 			)
 		)
+		(property "LCSC" "C6119795"
+			(at 182.88 58.42 0)
+			(effects
+				(font
+					(size 1.27 1.27)
+				)
+				(hide yes)
+			)
+		)
 		(pin "1"
 		)
@@
 			)
 		)
+		(property "LCSC" "C138687"
+			(at 349.25 64.77 0)
+			(effects
+				(font
+					(size 1.27 1.27)
+				)
+				(hide yes)
+			)
+		)
 		(pin "2"
 		)
@@
 			)
 		)
+		(property "LCSC" "C107031"
+			(at 199.39 99.06 0)
+			(effects
+				(font
+					(size 1.27 1.27)
+				)
+				(hide yes)
+			)
+		)
 		(pin "1"
 		)
@@
 			)
 		)
+		(property "LCSC" "C11537"
+			(at 193.04 80.01 0)
+			(effects
+				(font
+					(size 1.27 1.27)
+				)
+				(hide yes)
+			)
+		)
 		(pin "1"
 		)
@@
 			)
 		)
+		(property "LCSC" "C51205"
+			(at 311.15 64.77 0)
+			(effects
+				(font
+					(size 1.27 1.27)
+				)
+				(hide yes)
+			)
+		)
 		(pin "2"
 		)
@@
 			)
 		)
+		(property "LCSC" ""
+			(at 294.64 62.23 90)
+			(effects
+				(font
+					(size 1.27 1.27)
+				)
+				(hide yes)
+			)
+		)
 		(pin "4"
 		)
@@
 			)
 		)
+		(property "LCSC" "C138687"
+			(at 361.95 64.77 0)
+			(effects
+				(font
+					(size 1.27 1.27)
+				)
+				(hide yes)
+			)
+		)
 		(pin "2"
 		)
@@
 			)
 		)
+		(property "LCSC" "C138687"
+			(at 374.65 64.77 0)
+			(effects
+				(font
+					(size 1.27 1.27)
+				)
+				(hide yes)
+			)
+		)
 		(pin "2"
 		)
@@
 			)
 		)
+		(property "LCSC" "C114151"
+			(at 187.96 72.39 0)
+			(effects
+				(font
+					(size 1.27 1.27)
+				)
+				(hide yes)
+			)
+		)
 		(pin "1"
 		)
@@
 			)
 		)
+		(property "LCSC" "C25921"
+			(at 300.99 74.93 0)
+			(effects
+				(font
+					(size 1.27 1.27)
+				)
+				(hide yes)
+			)
+		)
 		(pin "1"
 		)
@@
 			)
 		)
+		(property "LCSC" "C51205"
+			(at 323.85 64.77 0)
+			(effects
+				(font
+					(size 1.27 1.27)
+				)
+				(hide yes)
+			)
+		)
 		(pin "2"
 		)
@@
 			)
 		)
+		(property "LCSC" "C51205"
+			(at 336.55 64.77 0)
+			(effects
+				(font
+					(size 1.27 1.27)
+				)
+				(hide yes)
+			)
+		)
 		(pin "2"
 		)
@@
 			(at 199.39 88.9 0)
 			(effects
+				(font
+					(size 1.27 1.27)
+				)
+				(hide yes)
+			)
+		)
+		(property "LCSC" "C25895"
+			(at 199.39 88.9 0)
+			(effects

Commit message: lcsc again
Parts:
- C100: LCSC (none) -> C107010
- C101: LCSC (none) -> C2932476
- C103, C113, C114: LCSC (none) -> C98192
- C105, C106: LCSC (none) -> C2762594
- C107: LCSC (none) -> C1525
- C108: LCSC (none) -> C15195
- C98: LCSC (none) -> C272875
- C99: LCSC (none) -> C106200
- R63: LCSC (none) -> C852768
- R64, R65: LCSC (none) -> C109318
- R66: LCSC (none) -> C185465
- R68, R70: LCSC (none) -> C852869
- R69, R71: LCSC (none) -> C6779318
- R72: LCSC (none) -> C60491
- R75: LCSC (none) -> C137983
- R76: LCSC (none) -> C185445
Changed lines of the file:
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@@
 			)
 		)
+		(property "LCSC" "C107010"
+			(at 55.88 203.2 0)
+			(effects
+				(font
+					(size 1.27 1.27)
+				)
+				(hide yes)
+			)
+		)
 		(pin "1"
 		)
@@
 			)
 		)
+		(property "LCSC" "C106200"
+			(at 29.21 203.2 0)
+			(effects
+				(font
+					(size 1.27 1.27)
+				)
+				(hide yes)
+			)
+		)
 		(pin "1"
 		)
@@
 			)
 		)
+		(property "LCSC" "C185445"
+			(at 55.88 254 0)
+			(effects
+				(font
+					(size 1.27 1.27)
+				)
+				(hide yes)
+			)
+		)
 		(pin "2"
 		)
@@
 		(on_board yes)
 		(dnp no)
-		(fields_autoplaced yes)
 		(property "Reference" "R75"
-			(at 162.56 184.15 90)
+			(at 162.56 185.674 90)
 			(effects
 				(font
@@
 		)
 		(property "Value" "40.2k"
-			(at 162.56 186.69 90)
+			(at 162.56 188.214 90)
 			(effects
 				(font
@@
 			)
 		)
+		(property "LCSC" "C137983"
+			(at 162.56 190.5 90)
+			(effects
+				(font
+					(size 1.27 1.27)
+				)
+				(hide yes)
+			)
+		)
 		(pin "2"
 		)
@@
 			)
 		)
+		(property "LCSC" "C2932476"
+			(at 187.96 177.8 0)
+			(effects
+				(font
+					(size 1.27 1.27)
+				)
+				(hide yes)
+			)
+		)
 		(pin "1"
 		)
@@
 			)
 		)
+		(property "LCSC" "C6779318"
+			(at 210.82 196.85 0)
+			(effects
+				(font
+					(size 1.27 1.27)
+				)
+				(hide yes)
+			)
+		)
 		(pin "1"
 		)
@@
 			)
 		)
+		(property "LCSC" "C852869"
+			(at 312.42 175.26 0)
+			(effects
+				(font
+					(size 1.27 1.27)
+				)
+				(hide yes)
+			)
+		)
 		(pin "1"
 		)
@@
 			)
 		)
+		(property "LCSC" "C1525"
+			(at 43.18 245.11 0)
+			(effects
+				(font
+					(size 1.27 1.27)
+				)
+				(hide yes)
+			)
+		)
 		(pin "2"
 		)
@@
 			)
 		)
+		(property "LCSC" "C98192"
+			(at 388.62 175.26 0)
+			(effects
+				(font
+					(size 1.27 1.27)
+				)
+				(hide yes)
+			)
+		)
 		(pin "1"
 		)
@@
 			)
 		)
+		(property "LCSC" "C109318"
+			(at 49.53 207.01 90)
+			(effects
+				(font
+					(size 1.27 1.27)
+				)
+				(hide yes)
+			)
+		)
 		(pin "2"
 		)
@@
 			)
 		)
+		(property "LCSC" "C109318"
+			(at 49.53 199.39 90)
+			(effects
+				(font
+					(size 1.27 1.27)
+				)
+				(hide yes)
+			)
+		)
 		(pin "2"
 		)
@@
 			)
 		)
+		(property "LCSC" "C6779318"
+			(at 312.42 185.42 0)
+			(effects
+				(font
+					(size 1.27 1.27)
+				)
+				(hide yes)
+			)
+		)
 		(pin "1"
 		)
@@
 		(dnp no)
 		(property "Reference" "R66"
-			(at 173.482 214.63 90)
+			(at 173.482 217.424 90)
 			(effects
 				(font
@@
 		)
 		(property "Value" "14.3k"
-			(at 177.8 212.344 90)
+			(at 174.498 212.344 90)
 			(effects
 				(font
@@
 			)
 		)
+		(property "LCSC" "C185465"
+			(at 171.45 214.63 90)
+			(effects
+				(font
+					(size 1.27 1.27)
+				)
+				(hide yes)
+			)
+		)
 		(pin "2"
 		)
@@
 			)
 		)
+		(property "LCSC" "C2762594"
+			(at 189.23 259.08 0)
+			(effects
+				(font
+					(size 1.27 1.27)
+				)
+				(hide yes)
+			)
+		)
 		(pin "1"
 		)
@@
 			)
 		)
+		(property "LCSC" "C98192"
+			(at 375.92 175.26 0)
+			(effects
+				(font
+					(size 1.27 1.27)
+				)
+				(hide yes)
+			)
+		)
 		(pin "1"
 		)
@@
 			)
 		)
+		(property "LCSC" "C60491"
+			(at 74.93 247.65 90)
+			(effects
+				(font
+					(size 1.27 1.27)
+				)
+				(hide yes)
+			)
+		)
 		(pin "1"
 		)
@@
 			)
 		)
+		(property "LCSC" "C852768"
+			(at 21.59 212.09 0)
+			(effects
+				(font
+					(size 1.27 1.27)
+				)
+				(hide yes)
+			)
+		)
 		(pin "1"
 		)
@@
 			)
 		)
+		(property "LCSC" "C272875"
+			(at 21.59 200.66 0)
+			(effects
+				(font
+					(size 1.27 1.27)
+				)
+				(hide yes)
+			)
+		)
 		(pin "1"
 		)
@@
 			)
 		)
+		(property "LCSC" "C2762594"
+			(at 203.2 260.35 0)
+			(effects
+				(font
+					(size 1.27 1.27)
+				)
+				(hide yes)
+			)
+		)
 		(pin "1"
 		)
@@
 			)
 		)
+		(property "LCSC" "C98192"
+			(at 363.22 175.26 0)
+			(effects
+				(font
+					(size 1.27 1.27)
+				)
+				(hide yes)
+			)
+		)
 		(pin "1"
 		)
@@
 			)
 		)
+		(property "LCSC" "C15195"
+			(at 85.09 257.81 0)
+			(effects
+				(font
+					(size 1.27 1.27)
+				)
+				(hide yes)
+			)
+		)
 		(pin "2"
 		)
@@
 			(at 210.82 184.15 0)
 			(effects
+				(font
+					(size 1.27 1.27)
+				)
+				(hide yes)
+			)
+		)
+		(property "LCSC" "C852869"
+			(at 210.82 184.15 0)
+			(effects
