File: MotorDriver.kicad_sch (KiCad schematic)
At the start: 1 part

Commit message: motor drivers done
Parts:
- removed U8: ~, symbol Dry_Lettuce:DRV8251DDAR
- added C64, C71: 1uf, Capacitor_SMD:C_0603_1608Metric, symbol Device:C
- added C65, C68: 0.1uf, Capacitor_SMD:C_0603_1608Metric, symbol Device:C
- added R32, R34: 100m, Resistor_SMD:R_1206_3216Metric, symbol Device:R
- added U13, U8: ~, Package_DFN_QFN:Maxim_TDFN-12-1EP_3x3mm_P0.5mm_EP1.7x2.5mm, symbol Dry_Lettuce:MAX14870IC
Connections:
- net DIR: now also U8.6 (DIR)
- net M1: now also U8.2 (M1)
- net M2: now also U8.11 (M2)
- net PWM: now also U8.5 (PWM)
- net VCC: now also C64.1, C65.1, U8.10 (VDD), U8.3 (VDD)
- new net: R32.1, U8.1 (COM), U8.12 (COM), U8.4 (SNS)
- new net: R34.1, U13.1 (COM), U13.12 (COM), U13.4 (SNS)
- new net +12V: C68.1, C71.1, U13.10 (VDD), U13.3 (VDD)
- new net FAULT: U8.7 (FAULT)
- new net GND: C64.2, C65.2, C68.2, C71.2, R32.2, R34.2, U13.8 (EN), U13.9 (GND), U8.8 (EN), U8.9 (GND)

Commit message: i think its fine?
@will-da-pro help
Parts:
- renumbered C65 to C1, C64 to C2, C68 to C3, C71 to C4, R32 to R1, R34 to R2, U8 to U1, U13 to U2
Changed lines of the file:
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@@
 		(on_board yes)
 		(dnp no)
-		(property "Reference" "C65"
+		(property "Reference" "C1"
 			(at 28.194 34.798 0)
 			(effects
@@
 				)
 			)
+			(project "MotorDriver"
+				(path "/48ed61e9-c240-49d3-9c03-d53f8f46ca65"
+					(reference "C1")
+					(unit 1)
+				)
+			)
 		)
 	)
@@
 		(on_board yes)
 		(dnp no)
-		(property "Reference" "#PWR059"
+		(property "Reference" "#PWR01"
 			(at 40.64 71.12 0)
 			(effects
@@
 				)
 			)
+			(project "MotorDriver"
+				(path "/48ed61e9-c240-49d3-9c03-d53f8f46ca65"
+					(reference "#PWR01")
+					(unit 1)
+				)
+			)
 		)
 	)
@@
 		(on_board yes)
 		(dnp no)
-		(property "Reference" "#PWR0100"
+		(property "Reference" "#PWR06"
 			(at 93.98 43.18 0)
 			(effects
@@
 				)
 			)
+			(project "MotorDriver"
+				(path "/48ed61e9-c240-49d3-9c03-d53f8f46ca65"
+					(reference "#PWR06")
+					(unit 1)
+				)
+			)
 		)
 	)
@@
 		(dnp no)
 		(fields_autoplaced yes)
-		(property "Reference" "#PWR058"
+		(property "Reference" "#PWR03"
 			(at 59.69 71.12 0)
 			(effects
@@
 				)
 			)
+			(project "MotorDriver"
+				(path "/48ed61e9-c240-49d3-9c03-d53f8f46ca65"
+					(reference "#PWR03")
+					(unit 1)
+				)
+			)
 		)
 	)
@@
 		(on_board yes)
 		(dnp no)
-		(property "Reference" "U8"
+		(property "Reference" "U1"
 			(at 64.516 51.816 0)
 			(effects
@@
 				)
 			)
+			(project "MotorDriver"
+				(path "/48ed61e9-c240-49d3-9c03-d53f8f46ca65"
+					(reference "U1")
+					(unit 1)
+				)
+			)
 		)
 	)
@@
 		(dnp no)
 		(fields_autoplaced yes)
-		(property "Reference" "#PWR098"
+		(property "Reference" "#PWR04"
 			(at 78.74 62.23 0)
 			(effects
@@
 				)
 			)
+			(project "MotorDriver"
+				(path "/48ed61e9-c240-49d3-9c03-d53f8f46ca65"
+					(reference "#PWR04")
+					(unit 1)
+				)
+			)
 		)
 	)
@@
 		(on_board yes)
 		(dnp no)
-		(property "Reference" "#PWR057"
+		(property "Reference" "#PWR02"
 			(at 46.99 45.72 0)
 			(effects
@@
 				)
 			)
+			(project "MotorDriver"
+				(path "/48ed61e9-c240-49d3-9c03-d53f8f46ca65"
+					(reference "#PWR02")
+					(unit 1)
+				)
+			)
 		)
 	)
@@
 		(on_board yes)
 		(dnp no)
-		(property "Reference" "C64"
+		(property "Reference" "C2"
 			(at 39.624 34.798 0)
 			(effects
@@
 				)
 			)
+			(project "MotorDriver"
+				(path "/48ed61e9-c240-49d3-9c03-d53f8f46ca65"
+					(reference "C2")
+					(unit 1)
+				)
+			)
 		)
 	)
@@
 		(on_board yes)
 		(dnp no)
-		(property "Reference" "C68"
+		(property "Reference" "C3"
 			(at 104.902 24.384 0)
 			(effects
@@
 				)
 			)
+			(project "MotorDriver"
+				(path "/48ed61e9-c240-49d3-9c03-d53f8f46ca65"
+					(reference "C3")
+					(unit 1)
+				)
+			)
 		)
 	)
@@
 		(on_board yes)
 		(dnp no)
-		(property "Reference" "#PWR099"
+		(property "Reference" "#PWR05"
 			(at 83.82 30.48 0)
 			(effects
@@
 				)
 			)
+			(project "MotorDriver"
+				(path "/48ed61e9-c240-49d3-9c03-d53f8f46ca65"
+					(reference "#PWR05")
+					(unit 1)
+				)
+			)
 		)
 	)
@@
 		(dnp no)
 		(fields_autoplaced yes)
-		(property "Reference" "#PWR0102"
+		(property "Reference" "#PWR07"
 			(at 104.14 31.75 0)
 			(effects
@@
 				)
 			)
+			(project "MotorDriver"
+				(path "/48ed61e9-c240-49d3-9c03-d53f8f46ca65"
+					(reference "#PWR07")
+					(unit 1)
+				)
+			)
 		)
 	)
@@
 		(on_board yes)
 		(dnp no)
-		(property "Reference" "C71"
+		(property "Reference" "C4"
 			(at 104.902 35.814 0)
 			(effects
@@
 				)
 			)
+			(project "MotorDriver"
+				(path "/48ed61e9-c240-49d3-9c03-d53f8f46ca65"
+					(reference "C4")
+					(unit 1)
+				)
+			)
 		)
 	)
@@
 		(on_board yes)
 		(dnp no)
-		(property "Reference" "U13"
+		(property "Reference" "U2"
 			(at 90.424 60.706 0)
 			(effects
@@
 				)
 			)
+			(project "MotorDriver"
+				(path "/48ed61e9-c240-49d3-9c03-d53f8f46ca65"
+					(reference "U2")
+					(unit 1)
+				)
+			)
 		)
 	)
@@
 		(on_board yes)
 		(dnp no)
-		(property "Reference" "R34"
+		(property "Reference" "R2"
 			(at 78.74 52.07 90)
 			(effects
@@
 				)
 			)
+			(project "MotorDriver"
+				(path "/48ed61e9-c240-49d3-9c03-d53f8f46ca65"
+					(reference "R2")
+					(unit 1)
+				)
+			)
 		)
 	)
@@
 		(on_board yes)
 		(dnp no)
-		(property "Reference" "R32"
+		(property "Reference" "R1"
 			(at 55.88 63.5 90)
 			(effects
@@
 				)
 			)
-		)
-	)
+			(project "MotorDriver"
+				(path "/48ed61e9-c240-49d3-9c03-d53f8f46ca65"
+					(reference "R1")
+					(unit 1)
+				)
+			)
+		)
+	)
+	(sheet_instances
+		(path "/"
+			(page "1")
+		)
+	)
+	(embedded_fonts no)
 )
