File: down_leds.kicad_sch (KiCad schematic)
At the start: 13 parts, among them U5 DMG2305UX-7

Commit message: switch now bigger
Connections:
- net +5V: now also U5.2 (S); no longer U5.3 (D)
- net DOWN_LED_DRAIN: now also U5.3 (D); no longer U5.2 (S)
Other:
- moved on the sheet: U5
Changed lines of the file:
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@@
 	(symbol
 		(lib_id "Transistor_FET:DMG2305UX-7")
-		(at 92.71 64.77 0)
-		(mirror y)
+		(at 92.71 64.77 180)
 		(unit 1)
 		(body_style 1)

Commit message: reinstated fixed battery schematic
Connections:
- net +5V: now also U5.3 (D); no longer U5.2 (S)
- net DOWN_LED_DRAIN: now also U5.2 (S); no longer U5.3 (D)
Other:
- moved on the sheet: U5
Changed lines of the file:
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@@
 	(symbol
 		(lib_id "Transistor_FET:DMG2305UX-7")
-		(at 92.71 64.77 180)
+		(at 92.71 64.77 0)
+		(mirror y)
 		(unit 1)
 		(body_style 1)
@@
 		(fields_autoplaced yes)
 		(property "Reference" "U5"
-			(at 86.36 64.77 90)
+			(at 87.63 63.4999 0)
 			(show_name no)
 			(do_not_autoplace no)
@@
 					(size 1.27 1.27)
 				)
+				(justify left)
 			)
 		)
 		(property "Value" "DMG2305UX-7"
-			(at 83.82 64.77 90)
+			(at 87.63 66.0399 0)
 			(show_name no)
 			(do_not_autoplace no)
@@
 					(size 1.27 1.27)
 				)
+				(justify left)
 			)
 		)
